File: Schematic/Addressing.sch (KiCad schematic (older format))
At the start: 5 parts, among them IC10 74LS593, IC11 74HCT251, IC7 74HCT574, IC8 74HCT574, IC9 74LS593

Commit message: Updated the schematic and also moved to KiCad 5.
Parts:
- IC10, IC9: symbol 74LS593 -> 74LS593:74LS593
- IC11: symbol 74LS251-RESCUE-Schematic -> Schematic-rescue:74LS251-RESCUE-Schematic
- IC7, IC8: symbol 74LS574-RESCUE-Schematic -> 74LS593:74LS574-RESCUE-Schematic
Connections:
- net Lo: now also IC9.14 (CCKEN#)
- net ~Clkbar: no longer IC9.13 (CCK)
- net at IC10.11 (RCO#): now also IC9.13 (CCK); no longer IC9.14 (CCKEN#)
Changed lines of the file:
@@
-EESchema Schematic File Version 2
-LIBS:Schematic-rescue
-LIBS:power
-LIBS:device
-LIBS:switches
-LIBS:relays
-LIBS:motors
-LIBS:transistors
-LIBS:conn
-LIBS:linear
-LIBS:regul
-LIBS:74xx
-LIBS:cmos4000
-LIBS:adc-dac
-LIBS:memory
-LIBS:xilinx
-LIBS:microcontrollers
-LIBS:dsp
-LIBS:microchip
-LIBS:analog_switches
-LIBS:motorola
-LIBS:texas
-LIBS:intel
-LIBS:audio
-LIBS:interface
-LIBS:digital-audio
-LIBS:philips
-LIBS:display
-LIBS:cypress
-LIBS:siliconi
-LIBS:opto
-LIBS:atmel
-LIBS:contrib
-LIBS:valves
-LIBS:M27C322-100F1
-LIBS:74LS574
-LIBS:AT27C1024-70PU
-LIBS:QX14T50B1.843200B50TT
-LIBS:SN74LS273NE4
-LIBS:UM245R
-LIBS:7400-ic
-LIBS:74LS593
-LIBS:74LS139
+EESchema Schematic File Version 4
 LIBS:Schematic-cache
-EELAYER 25 0
+EELAYER 29 0
 EELAYER END
 $Descr A4 11693 8268
@@
 Jump\nLogic
 $Comp
-L GNDREF #PWR014
+L power:GNDREF #PWR014
 U 1 1 5C911F8E
 P 6950 6050
@@
 $EndComp
 $Comp
-L VCC #PWR015
+L power:VCC #PWR015
 U 1 1 5C911FB4
 P 6950 5850
@@
 $EndComp
 $Comp
-L 74LS574-RESCUE-Schematic IC7
+L 74LS593:74LS574-RESCUE-Schematic IC7
 U 1 1 5C98EE54
 P 3000 1750
@@
 $EndComp
 $Comp
-L 74LS574-RESCUE-Schematic IC8
+L 74LS593:74LS574-RESCUE-Schematic IC8
 U 1 1 5C98FD7B
 P 2950 3700
@@
 	1    0    0    -1
 $EndComp
-Wire Bus Line
-	4000 650  4000 3800
 Entry Wire Line
 	3900 3900 4000 3800
@@
 	1950 2050 2050 1950
 Wire Bus Line
-	1950 1350 1950 4900
-Wire Bus Line
 	1950 4900 1200 4900
 Entry Wire Line
@@
 d7
 $Comp
-L VCC #PWR016
+L power:VCC #PWR016
 U 1 1 5C99A807
 P 3850 2150
@@
 $EndComp
 $Comp
-L VCC #PWR017
+L power:VCC #PWR017
 U 1 1 5C99A830
 P 3850 4100
@@
 $EndComp
 $Comp
-L GNDREF #PWR018
+L power:GNDREF #PWR018
 U 1 1 5C99A88B
 P 3850 2250
@@
 $EndComp
 $Comp
-L GNDREF #PWR019
+L power:GNDREF #PWR019
 U 1 1 5C99AB18
 P 3850 4200
@@
 	2300 2250 2100 2250
 Wire Wire Line
-	2100 2250 2100 5400
+	2100 2250 2100 4200
 Wire Wire Line
 	2250 4200 2100 4200
@@
 	2250 4450 2550 4450
 $Comp
-L 74LS593 IC9
+L 74LS593:74LS593 IC9
 U 1 1 5C99FB31
 P 6350 1700
@@
 $EndComp
 $Comp
-L 74LS593 IC10
+L 74LS593:74LS593 IC10
 U 1 1 5C99FFFA
 P 6350 3650
@@
 	7000 3200 7050 3200
 Wire Wire Line
-	7050 3200 7050 2150
-Wire Wire Line
-	7050 2150 7000 2150
-Wire Wire Line
-	4950 4100 5650 4100
+	4950 4100 5350 4100
 Entry Wire Line
 	4000 3800 4100 3900
 Wire Wire Line
 	5650 3900 4100 3900
-Wire Wire Line
-	4800 2150 5650 2150
-$Comp
-L VCC #PWR020
+$Comp
+L power:VCC #PWR020
 U 1 1 5C9A1A2E
 P 8550 1300
@@
 NoConn ~ 7000 1250
 $Comp
-L GNDREF #PWR021
+L power:GNDREF #PWR021
 U 1 1 5C9A1C76
 P 8550 3650
@@
 $EndComp
 $Comp
-L GNDREF #PWR022
+L power:GNDREF #PWR022
 U 1 1 5C9A1E6F
 P 8550 1700
@@
 ~ARena
 $Comp
-L VCC #PWR023
+L power:VCC #PWR023
 U 1 1 5C9A2F13
 P 8550 3250
@@
 ~Reset
 $Comp
-L 74LS251-RESCUE-Schematic U?
+L Schematic-rescue:74LS251-RESCUE-Schematic U?
 U 1 1 5CA1932F
 P 6150 5400
@@
 Wire Bus Line
 	4250 5500 4500 5500
-Wire Bus Line
-	4500 5500 4500 5750
 Entry Wire Line
 	4500 5750 4600 5850
@@
 	7000 4000 7300 4000
 Wire Wire Line
-	7000 3400 7300 3400
-Wire Wire Line
-	7000 1450 7250 1450
+	7000 3400 7100 3400
+Wire Wire Line
+	7000 1450 7150 1450
 Wire Wire Line
 	7000 1350 7800 1350
@@
 Text GLabel 7300 3800 2    60   Input ~ 0
 PCincr
-Text GLabel 4800 2150 0    60   Input ~ 0
+Text GLabel 5200 2050 0    60   Input ~ 0
 ~Clkbar
 NoConn ~ 6850 4900
@@
 Hi
 Wire Wire Line
-	5200 2050 5200 2150
-Connection ~ 5200 2150
-Wire Wire Line
 	5350 4000 5350 4100
 Connection ~ 5350 4100
@@
 Connection ~ 7100 3400
 Wire Wire Line
-	7150 1850 7150 1450
+	7150 1850 7150 1750
 Connection ~ 7150 1450
 Wire Wire Line
 	7000 1750 7150 1750
 Connection ~ 7150 1750
+Wire Wire Line
+	2100 4200 2100 5400
+Wire Wire Line
+	5350 4100 5650 4100
+Wire Wire Line
+	7100 3400 7300 3400
+Wire Wire Line
+	7150 1450 7250 1450
+Wire Wire Line
+	7150 1750 7150 1450
+Wire Wire Line
+	7150 2150 7150 1850
+Wire Wire Line
+	7000 2150 7150 2150
+Connection ~ 7150 1850
+Wire Wire Line
+	5650 2150 5650 2550
+Wire Wire Line
+	5650 2550 7050 2550
+Wire Wire Line
+	7050 2550 7050 3200
+Wire Bus Line
+	4500 5500 4500 5750
+Wire Bus Line
+	4000 650  4000 3800
+Wire Bus Line
+	1950 1350 1950 4900
 $EndSCHEMATC
