File: Schematic/MemoryIO.sch (KiCad schematic (older format))
At the start: 4 parts, among them IC1 HM62256BLP-7, IC15 74LS139, IC2 28C256, IC3 UM245R

Commit message: Fixed up some schematic DCN mistakes and also a few minor typos and diagram issues.
Connections:
- net labels added: adr[0..15], d[0..7]
- net labels removed: AddressBus, DataBus
- wire segments 81 -> 84
Other:
- note added: "AddressBus"
- note added: "DataBus"
Changed lines of the file:
@@
 Wire Bus Line
 	2100 4550 3400 4550
-Text GLabel 2100 4550 0    60   Input ~ 0
-AddressBus
 Entry Wire Line
 	6650 1050 6750 950
@@
 Wire Bus Line
 	6750 850  9800 850
-Text GLabel 9800 850  2    60   Input ~ 0
-DataBus
 Wire Wire Line
 	5100 1050 6650 1050
@@
 adr15
 $Comp
-L GNDREF #PWR?
+L GNDREF #PWR09
 U 1 1 5C9A4A6B
-P 3750 6000
-F 0 "#PWR?" H 3750 5750 50  0001 C CNN
-F 1 "GNDREF" H 3750 5850 50  0000 C CNN
-F 2 "" H 3750 6000 50  0001 C CNN
-F 3 "" H 3750 6000 50  0001 C CNN
-	1    3750 6000
+P 3750 6200
+F 0 "#PWR09" H 3750 5950 50  0001 C CNN
+F 1 "GNDREF" H 3750 6050 50  0000 C CNN
+F 2 "" H 3750 6200 50  0001 C CNN
+F 3 "" H 3750 6200 50  0001 C CNN
+	1    3750 6200
 	1    0    0    -1
 $EndComp
@@
 	3850 5500 3750 5500
 Wire Wire Line
-	3750 5500 3750 6000
-Wire Wire Line
-	3750 6000 3850 6000
+	3750 5500 3750 6200
 NoConn ~ 5550 5450
 NoConn ~ 5550 5850
@@
 Text Notes 4550 5750 0    60   ~ 0
 Inverter
-Text Notes 3900 6450 0    60   ~ 0
+Text Notes 3900 6700 0    60   ~ 0
 Rather than add one more chip to the\ndesign, we use this demux as an inverter
 Wire Wire Line
@@
 Wire Wire Line
 	3850 4650 3850 4550
+Text GLabel 2100 4550 0    60   Input ~ 0
+adr[0..15]
+Text GLabel 9800 850  2    60   Input ~ 0
+d[0..7]
+Text Notes 2450 4500 0    60   ~ 0
+AddressBus
+Text Notes 7050 800  0    60   ~ 0
+DataBus
+Wire Wire Line
+	3950 6100 3750 6100
+Connection ~ 3750 6100
+$Comp
+L VCC #PWR010
+U 1 1 5C9AF8FD
+P 3400 5900
+F 0 "#PWR010" H 3400 5750 50  0001 C CNN
+F 1 "VCC" H 3400 6050 50  0000 C CNN
+F 2 "" H 3400 5900 50  0001 C CNN
+F 3 "" H 3400 5900 50  0001 C CNN
+	1    3400 5900
+	1    0    0    -1
+$EndComp
+Wire Wire Line
+	3850 5800 3750 5800
+Connection ~ 3750 5800
+Wire Wire Line
+	3950 6000 3400 6000
+Wire Wire Line
+	3400 6000 3400 5900
 $EndSCHEMATC

Commit message: Generated a new schematic of the circuit
Parts:
- IC15: symbol 74LS139 -> 74LS139-RESCUE-Schematic
Changed lines of the file:
@@
 EESchema Schematic File Version 2
+LIBS:Schematic-rescue
 LIBS:power
 LIBS:device
@@
 LIBS:7400-ic
 LIBS:74LS593
+LIBS:74LS139
 LIBS:Schematic-cache
 EELAYER 25 0
@@
 	5200 4750 5300 4750
 $Comp
-L 74LS139 IC15
+L 74LS139-RESCUE-Schematic IC15
 U 2 1 5C9A3AED
 P 4700 5750
+AR Path="/5C9A3AED" Ref="IC15"  Part="2"
+AR Path="/5C984F41/5C9A3AED" Ref="IC15"  Part="2"
 F 0 "IC15" H 4700 6300 50  0000 C CNN
 F 1 "74LS139" H 4700 6200 50  0000 C CNN
@@
 Text Notes 7050 800  0    60   ~ 0
 DataBus
-Wire Wire Line
-	3950 6100 3750 6100
 Connection ~ 3750 6100
+Wire Wire Line
+	3850 5800 3750 5800
+Connection ~ 3750 5800
+Wire Wire Line
+	3400 6000 3400 5900
 $Comp
 L VCC #PWR010
@@
 $EndComp
 Wire Wire Line
-	3850 5800 3750 5800
-Connection ~ 3750 5800
-Wire Wire Line
 	3950 6000 3400 6000
 Wire Wire Line
-	3400 6000 3400 5900
+	3950 6100 3750 6100
 $EndSCHEMATC

Commit message: Working on the PCB
Parts:
- IC1: footprint DIP28 -> Housings_DIP:DIP-28_W7.62mm_Socket
- IC15: footprint (none) -> Housings_DIP:DIP-16_W7.62mm_Socket
- IC2: footprint (none) -> Housings_DIP:DIP-28_W15.24mm_Socket
- IC3: footprint DIPS1500W50P254L3300H1050Q24N -> Housings_DIP:DIP-24_W7.62mm_Socket
Changed lines of the file:
@@
 F 0 "IC1" H 4600 2800 50  0000 C CNN
 F 1 "HM62256BLP-7" H 4550 2700 50  0000 C CNN
-F 2 "DIP28" H 4600 1800 50  0001 C CIN
+F 2 "Housings_DIP:DIP-28_W7.62mm_Socket" H 4600 1800 50  0001 C CIN
 F 3 "" H 4600 1800 50  0001 C CNN
 	1    4600 1800
@@
 F 0 "IC3" H 8550 1900 50  0000 L CNN
 F 1 "UM245R" H 8450 1800 50  0000 L CNN
-F 2 "DIPS1500W50P254L3300H1050Q24N" H 9000 1700 50  0001 L CNN
+F 2 "Housings_DIP:DIP-24_W7.62mm_Socket" H 9000 1700 50  0001 L CNN
 F 3 "http://www.ftdichip.com/Support/Documents/DataSheets/Modules/DS_UM245R.pdf" H 9000 1600 50  0001 L CNN
 F 4 "Interface Development Tools USB to Parallel FIFO Dev Mod for FT245R" H 9000 1500 50  0001 L CNN "Description"
@@
 F 0 "IC2" H 4600 4950 50  0000 C CNN
 F 1 "28C256" H 4600 4850 50  0000 C CNN
-F 2 "" H 4600 3850 50  0001 C CNN
+F 2 "Housings_DIP:DIP-28_W15.24mm_Socket" H 4600 3850 50  0001 C CNN
 F 3 "" H 4600 3850 50  0001 C CNN
 	1    4600 3850
@@
 F 0 "IC15" H 4700 6300 50  0000 C CNN
 F 1 "74LS139" H 4700 6200 50  0000 C CNN
-F 2 "" H 4700 5750 50  0001 C CNN
+F 2 "Housings_DIP:DIP-16_W7.62mm_Socket" H 4700 5750 50  0001 C CNN
 F 3 "" H 4700 5750 50  0001 C CNN
 	2    4700 5750

Commit message: Brought the schematic and PCB board design up to date.
Parts:
- removed IC15: 74LS139, Housings_DIP:DIP-16_W7.62mm_Socket, symbol 74LS139-RESCUE-Schematic
- added IC17: 74LS04, Housings_DIP:DIP-14_W7.62mm_Socket, symbol 74LS04
- IC1: value HM62256BLP-7 -> AS6C62256; footprint Housings_DIP:DIP-28_W7.62mm_Socket -> Housings_DIP:DIP-28_W15.24mm_Socket
- IC3: footprint Housings_DIP:DIP-24_W7.62mm_Socket -> Housings_DIP:DIP-24_W15.24mm_Socket
Connections:
- net VCC: now also IC17.14 (VCC); no longer IC2.27 (~WE)
- net adr15: now also IC17.13
- net at IC1.20 (~CS): now also IC17.12
- net ~TXready: now reaches IC3.22 (TEX#)
- net ~RXready: now reaches IC3.23 (RXF#)
- net IOload renamed ~IOload
- net MEMload renamed ~MEMload
- net MEMresult renamed ~MEMresult
- net UARTresult renamed ~UARTresult
- new net GND: IC17.7 (GND)
- new net Hi: IC2.27 (~WE)
- no-connect marks 13 -> 8
Other:
- note added: "The RAM and ROM components are 32Kbytes\neach. The adr15 line is inverted so that ROM\noccupies the lower 32K of the address space,\nand RAM in the upper 32K. Both output to the\ndata bus, controlled by the MEMresult line."
- note added: "The UART is also connected to the\ndata bus, and it has separate output\nand input control lines. There are two\nready lines which are sent to the Jump\nlogic."
- note removed: "Inverter"
- note removed: "Rather than add one more chip to the\ndesign, we use this demux as an inverter"
Changed lines of the file:
@@
 P 4600 1800
 F 0 "IC1" H 4600 2800 50  0000 C CNN
-F 1 "HM62256BLP-7" H 4550 2700 50  0000 C CNN
-F 2 "Housings_DIP:DIP-28_W7.62mm_Socket" H 4600 1800 50  0001 C CIN
+F 1 "AS6C62256" H 4600 2700 50  0000 C CNN
+F 2 "Housings_DIP:DIP-28_W15.24mm_Socket" H 4600 1800 50  0001 C CIN
 F 3 "" H 4600 1800 50  0001 C CNN
 	1    4600 1800
@@
 F 0 "IC3" H 8550 1900 50  0000 L CNN
 F 1 "UM245R" H 8450 1800 50  0000 L CNN
-F 2 "Housings_DIP:DIP-24_W7.62mm_Socket" H 9000 1700 50  0001 L CNN
+F 2 "Housings_DIP:DIP-24_W15.24mm_Socket" H 9000 1700 50  0001 L CNN
 F 3 "http://www.ftdichip.com/Support/Documents/DataSheets/Modules/DS_UM245R.pdf" H 9000 1600 50  0001 L CNN
 F 4 "Interface Development Tools USB to Parallel FIFO Dev Mod for FT245R" H 9000 1500 50  0001 L CNN "Description"
@@
 NoConn ~ 9150 1800
 NoConn ~ 9150 1900
-NoConn ~ 9150 2000
-NoConn ~ 9150 2100
 NoConn ~ 9150 2200
 NoConn ~ 9150 2300
@@
 NoConn ~ 7950 2600
 Text GLabel 7400 2500 0    60   Input ~ 0
-UARTresult
+~UARTresult
 Wire Wire Line
 	7400 2500 7950 2500
 Text GLabel 7200 2400 0    60   Input ~ 0
-IOload
+~IOload
 Wire Wire Line
 	7200 2400 7950 2400
 Text GLabel 6150 2000 2    60   Input ~ 0
-MEMload
+~MEMload
 Wire Wire Line
 	5100 2000 6150 2000
 Text GLabel 6100 1900 2    60   Input ~ 0
-MEMresult
+~MEMresult
 Wire Wire Line
 	5100 1900 6100 1900
-$Comp
-L VCC #PWR04
-U 1 1 5C997F19
-P 3850 4550
-F 0 "#PWR04" H 3850 4400 50  0001 C CNN
-F 1 "VCC" H 3850 4700 50  0000 C CNN
-F 2 "" H 3850 4550 50  0001 C CNN
-F 3 "" H 3850 4550 50  0001 C CNN
-	1    3850 4550
-	1    0    0    -1
-$EndComp
 Entry Wire Line
 	2250 4550 2350 4650
-Text Label 3550 4750 0    60   ~ 0
+Text Label 3300 4750 0    60   ~ 0
 adr15
 Text Notes 4500 1750 0    60   ~ 0
@@
 UART
 $Comp
-L GNDREF #PWR05
+L GNDREF #PWR04
 U 1 1 5C999C9E
 P 5250 2450
-F 0 "#PWR05" H 5250 2200 50  0001 C CNN
+F 0 "#PWR04" H 5250 2200 50  0001 C CNN
 F 1 "GNDREF" H 5250 2300 50  0000 C CNN
 F 2 "" H 5250 2450 50  0001 C CNN
@@
 $EndComp
 $Comp
-L VCC #PWR06
+L VCC #PWR05
 U 1 1 5C999CBE
 P 5250 2350
-F 0 "#PWR06" H 5250 2200 50  0001 C CNN
+F 0 "#PWR05" H 5250 2200 50  0001 C CNN
 F 1 "VCC" H 5250 2500 50  0000 C CNN
 F 2 "" H 5250 2350 50  0001 C CNN
@@
 $EndComp
 $Comp
-L GNDREF #PWR07
+L GNDREF #PWR06
 U 1 1 5C99A4F7
 P 5300 4750
-F 0 "#PWR07" H 5300 4500 50  0001 C CNN
+F 0 "#PWR06" H 5300 4500 50  0001 C CNN
 F 1 "GNDREF" H 5300 4600 50  0000 C CNN
 F 2 "" H 5300 4750 50  0001 C CNN
@@
 $EndComp
 $Comp
-L VCC #PWR08
+L VCC #PWR07
 U 1 1 5C99A542
 P 5300 4650
-F 0 "#PWR08" H 5300 4500 50  0001 C CNN
+F 0 "#PWR07" H 5300 4500 50  0001 C CNN
 F 1 "VCC" H 5300 4800 50  0000 C CNN
 F 2 "" H 5300 4650 50  0001 C CNN
@@
 Wire Wire Line
 	5200 4750 5300 4750
-$Comp
-L 74LS139-RESCUE-Schematic IC15
-U 2 1 5C9A3AED
-P 4700 5750
-AR Path="/5C9A3AED" Ref="IC15"  Part="2"
-AR Path="/5C984F41/5C9A3AED" Ref="IC15"  Part="2"
-F 0 "IC15" H 4700 6300 50  0000 C CNN
-F 1 "74LS139" H 4700 6200 50  0000 C CNN
-F 2 "Housings_DIP:DIP-16_W7.62mm_Socket" H 4700 5750 50  0001 C CNN
-F 3 "" H 4700 5750 50  0001 C CNN
-	2    4700 5750
-	1    0    0    -1
-$EndComp
 Wire Wire Line
 	2450 4750 3900 4750
 Wire Wire Line
 	2450 4750 2350 4650
-Wire Wire Line
-	3850 5650 2700 5650
-Wire Wire Line
-	2700 5650 2700 4750
 Connection ~ 2700 4750
-Text Label 3400 5650 0    60   ~ 0
+Text Label 3300 5300 0    60   ~ 0
 adr15
-$Comp
-L GNDREF #PWR09
-U 1 1 5C9A4A6B
-P 3750 6200
-F 0 "#PWR09" H 3750 5950 50  0001 C CNN
-F 1 "GNDREF" H 3750 6050 50  0000 C CNN
-F 2 "" H 3750 6200 50  0001 C CNN
-F 3 "" H 3750 6200 50  0001 C CNN
-	1    3750 6200
-	1    0    0    -1
-$EndComp
-Wire Wire Line
-	3850 5500 3750 5500
-Wire Wire Line
-	3750 5500 3750 6200
-NoConn ~ 5550 5450
-NoConn ~ 5550 5850
-NoConn ~ 5550 6050
-Text Notes 4550 5750 0    60   ~ 0
-Inverter
-Text Notes 3900 6700 0    60   ~ 0
-Rather than add one more chip to the\ndesign, we use this demux as an inverter
 Wire Wire Line
 	5100 2150 5700 2150
-Wire Wire Line
-	5700 2150 5700 5650
-Wire Wire Line
-	5700 5650 5550 5650
 Wire Wire Line
 	5950 1900 5950 4050
@@
 Wire Wire Line
 	3900 4650 3850 4650
-Wire Wire Line
-	3850 4650 3850 4550
 Text GLabel 2100 4550 0    60   Input ~ 0
 adr[0..15]
-Text GLabel 9800 850  2    60   Input ~ 0
+Text GLabel 9800 850  2    60   BiDi ~ 0
 d[0..7]
 Text Notes 2450 4500 0    60   ~ 0
@@
 Text Notes 7050 800  0    60   ~ 0
 DataBus
-Connection ~ 3750 6100
-Wire Wire Line
-	3850 5800 3750 5800
-Connection ~ 3750 5800
-Wire Wire Line
-	3400 6000 3400 5900
-$Comp
-L VCC #PWR010
-U 1 1 5C9AF8FD
-P 3400 5900
-F 0 "#PWR010" H 3400 5750 50  0001 C CNN
-F 1 "VCC" H 3400 6050 50  0000 C CNN
-F 2 "" H 3400 5900 50  0001 C CNN
-F 3 "" H 3400 5900 50  0001 C CNN
-	1    3400 5900
-	1    0    0    -1
-$EndComp
-Wire Wire Line
-	3950 6000 3400 6000
-Wire Wire Line
-	3950 6100 3750 6100
+Text GLabel 9350 2100 2    60   Output ~ 0
+~TXready
+Text GLabel 9350 2000 2    60   Output ~ 0
+~RXready
+Wire Wire Line
+	9150 2000 9350 2000
+Wire Wire Line
+	9150 2100 9350 2100
+Text GLabel 3850 4650 0    60   Input ~ 0
+Hi
+Text Notes 600  1200 0    60   ~ 0
+The RAM and ROM components are 32Kbytes\neach. The adr15 line is inverted so that ROM\noccupies the lower 32K of the address space,\nand RAM in the upper 32K. Both output to the\ndata bus, controlled by the MEMresult line.
+Text Notes 600  1800 0    60   ~ 0
+The UART is also connected to the\ndata bus, and it has separate output\nand input control lines.  There are two\nready lines which are sent to the Jump\nlogic.
+$Comp
+L 74LS04 IC17
+U 6 1 5CA2F410
+P 4600 5300
+F 0 "IC17" H 4795 5415 50  0000 C CNN
+F 1 "74LS04" H 4790 5175 50  0000 C CNN
+F 2 "Housings_DIP:DIP-14_W7.62mm_Socket" H 4600 5300 50  0001 C CNN
+F 3 "" H 4600 5300 50  0001 C CNN
+	6    4600 5300
+	1    0    0    -1
+$EndComp
+Wire Wire Line
+	4150 5300 2700 5300
+Wire Wire Line
+	2700 5300 2700 4750
+Wire Wire Line
+	5700 2150 5700 5300
+Wire Wire Line
+	5700 5300 5050 5300
 $EndSCHEMATC

Commit message: Updated the schematic and also moved to KiCad 5.
Parts:
- IC1: symbol HM62256BLP-7 -> memory:HM62256BLP-7
- IC17: value 74LS04 -> 74HCT04; symbol 74LS04 -> 74xx:74LS04
- IC2: symbol 28C256 -> memory:28C256
- IC3: symbol UM245R -> UM245R:UM245R
Connections:
- net VCC: no longer IC17.14 (VCC)
- removed net GND: IC17.7 (GND)
Changed lines of the file:
@@
-EESchema Schematic File Version 2
-LIBS:Schematic-rescue
-LIBS:power
-LIBS:device
-LIBS:switches
-LIBS:relays
-LIBS:motors
-LIBS:transistors
-LIBS:conn
-LIBS:linear
-LIBS:regul
-LIBS:74xx
-LIBS:cmos4000
-LIBS:adc-dac
-LIBS:memory
-LIBS:xilinx
-LIBS:microcontrollers
-LIBS:dsp
-LIBS:microchip
-LIBS:analog_switches
-LIBS:motorola
-LIBS:texas
-LIBS:intel
-LIBS:audio
-LIBS:interface
-LIBS:digital-audio
-LIBS:philips
-LIBS:display
-LIBS:cypress
-LIBS:siliconi
-LIBS:opto
-LIBS:atmel
-LIBS:contrib
-LIBS:valves
-LIBS:M27C322-100F1
-LIBS:74LS574
-LIBS:AT27C1024-70PU
-LIBS:QX14T50B1.843200B50TT
-LIBS:SN74LS273NE4
-LIBS:UM245R
-LIBS:7400-ic
-LIBS:74LS593
-LIBS:74LS139
+EESchema Schematic File Version 4
 LIBS:Schematic-cache
-EELAYER 25 0
+EELAYER 29 0
 EELAYER END
 $Descr A4 11693 8268
@@
 $EndDescr
 $Comp
-L HM62256BLP-7 IC1
+L memory:HM62256BLP-7 IC1
 U 1 1 5C997E5D
 P 4600 1800
@@
 Text Label 3550 4350 0    60   ~ 0
 adr14
-Wire Bus Line
-	3400 4550 3400 1150
-Wire Bus Line
-	2100 4550 3400 4550
 Entry Wire Line
 	6650 1050 6750 950
@@
 Entry Wire Line
 	6650 3650 6750 3550
-Wire Bus Line
-	6750 850  6750 3550
 Wire Bus Line
 	6750 850  9800 850
@@
 d7
 $Comp
-L UM245R IC3
+L UM245R:UM245R IC3
 U 1 1 5C998F7D
 P 7950 1600
@@
 Text Label 7700 2300 0    60   ~ 0
 d7
-Wire Bus Line
-	7550 850  7550 2200
-$Comp
-L GNDREF #PWR01
+$Comp
+L power:GNDREF #PWR01
 U 1 1 5C99C363
 P 7750 2700
@@
 $EndComp
 $Comp
-L GNDREF #PWR02
+L power:GNDREF #PWR02
 U 1 1 5C99C37E
 P 9350 2700
@@
 	9150 2700 9350 2700
 $Comp
-L VCC #PWR03
+L power:VCC #PWR03
 U 1 1 5C99C414
 P 9350 1500
@@
 	9350 1700 9150 1700
 Wire Wire Line
-	9350 1500 9350 1700
+	9350 1500 9350 1600
 Wire Wire Line
 	9150 1600 9350 1600
@@
 ~MEMresult
 Wire Wire Line
-	5100 1900 6100 1900
+	5100 1900 5950 1900
 Entry Wire Line
 	2250 4550 2350 4650
@@
 UART
 $Comp
-L GNDREF #PWR04
+L power:GNDREF #PWR04
 U 1 1 5C999C9E
 P 5250 2450
@@
 $EndComp
 $Comp
-L VCC #PWR05
+L power:VCC #PWR05
 U 1 1 5C999CBE
 P 5250 2350
@@
 	5200 2450 5250 2450
 $Comp
-L 28C256 IC2
+L memory:28C256 IC2
 U 1 1 5C99A013
 P 4600 3850
@@
 $EndComp
 $Comp
-L GNDREF #PWR06
+L power:GNDREF #PWR06
 U 1 1 5C99A4F7
 P 5300 4750
@@
 $EndComp
 $Comp
-L VCC #PWR07
+L power:VCC #PWR07
 U 1 1 5C99A542
 P 5300 4650
@@
 	5200 4750 5300 4750
 Wire Wire Line
-	2450 4750 3900 4750
+	2450 4750 2700 4750
 Wire Wire Line
 	2450 4750 2350 4650
@@
 The UART is also connected to the\ndata bus, and it has separate output\nand input control lines.  There are two\nready lines which are sent to the Jump\nlogic.
 $Comp
-L 74LS04 IC17
+L 74xx:74LS04 IC17
 U 6 1 5CA2F410
 P 4600 5300
 F 0 "IC17" H 4795 5415 50  0000 C CNN
-F 1 "74LS04" H 4790 5175 50  0000 C CNN
+F 1 "74HCT04" H 4790 5175 50  0000 C CNN
 F 2 "Housings_DIP:DIP-14_W7.62mm_Socket" H 4600 5300 50  0001 C CNN
 F 3 "" H 4600 5300 50  0001 C CNN
@@
 $EndComp
 Wire Wire Line
-	4150 5300 2700 5300
-Wire Wire Line
 	2700 5300 2700 4750
 Wire Wire Line
 	5700 2150 5700 5300
 Wire Wire Line
-	5700 5300 5050 5300
+	9350 1600 9350 1700
+Wire Wire Line
+	2700 4750 3900 4750
+Wire Wire Line
+	5950 1900 6100 1900
+Wire Wire Line
+	2700 5300 4300 5300
+Wire Wire Line
+	4900 5300 5700 5300
+Wire Bus Line
+	2100 4550 3400 4550
+Wire Bus Line
+	7550 850  7550 2200
+Wire Bus Line
+	6750 850  6750 3550
+Wire Bus Line
+	3400 1150 3400 4550
 $EndSCHEMATC
