File: Schematic/Schematic.kicad_pcb (KiCad board)
At the start: 2 copper layers, 234.9 x 114.3 mm, 41 parts, among them IC1 HM62256BLP-7, IC10 74LS593, IC11 74LS153, IC12 74LS574, IC13 74LS161-wkt, IC14 AT27C1024-70PU, IC15 74LS139, IC16 74LS138, IC2 28C256, IC3 UM245R, IC4 74LS574, IC5 74LS574, IC6 M27C322-100F1, IC7 74LS574, IC8 74LS574, IC9 74LS593, J1 GS3, SW1 SW_Push_Dual, SW2 SW_Push_Dual, U1 QX14T50B3.6864

Commit message: Brought the schematic and PCB board design up to date.
Parts:
- removed C2: 10uF, Capacitors_THT:CP_Radial_D5.0mm_P2.50mm
- added C20: 0.1uF, Capacitors_THT:C_Disc_D4.7mm_W2.5mm_P5.00mm, F.Cu at (116.3, 102.6)
- added C21: 0.1uF, Capacitors_THT:C_Disc_D4.7mm_W2.5mm_P5.00mm, F.Cu at (128.5, 106.7)
- added C22: 0.1uF, Capacitors_THT:C_Disc_D4.7mm_W2.5mm_P5.00mm, F.Cu at (94.0, 109.2)
- added D1: 1N4148, Diodes_THT:D_DO-35_SOD27_P2.54mm_Vertical_AnodeUp, F.Cu at (99.6, 111.8)
- added IC17: 74LS04, Housings_DIP:DIP-14_W7.62mm_Socket, F.Cu at (143.8, 76.7)
- added IC18: NE555, Housings_DIP:DIP-8_W7.62mm_Socket, F.Cu at (109.7, 107.2)
- added J2: DataBus Pin Header, Socket_Strips:Socket_Strip_Straight_1x10_Pitch2.54mm, F.Cu at (155.4, 39.1)
- added J3: AddressBus Pin Header, Socket_Strips:Socket_Strip_Straight_1x18_Pitch2.54mm, F.Cu at (25.4, 90.9)
- added J4: uSeq Pin Header, Socket_Strips:Socket_Strip_Straight_1x06_Pitch2.54mm, F.Cu at (246.4, 99.6)
- added J5: IR Pin Header, Socket_Strips:Socket_Strip_Straight_1x10_Pitch2.54mm, F.Cu at (235.7, 39.1)
- added R4: 1M, Resistors_THT:R_Axial_DIN0204_L3.6mm_D1.6mm_P1.90mm_Vertical, F.Cu at (121.9, 106.7)
- added R5: 10K, Resistors_THT:R_Axial_DIN0204_L3.6mm_D1.6mm_P1.90mm_Vertical, F.Cu at (104.6, 111.3)
- added R6: 10K, Resistors_THT:R_Axial_DIN0204_L3.6mm_D1.6mm_P1.90mm_Vertical, F.Cu at (104.6, 115.3)
- C1: footprint Capacitors_THT:CP_Radial_D5.0mm_P2.50mm -> Capacitors_THT:CP_Radial_D5.0mm_P2.00mm
- C10, C11, C12, C13, C14, C15, C16, C17, C18, C19, C4, C5, C6, C7, C8, C9: footprint Capacitors_THT:C_Disc_D3.0mm_W1.6mm_P2.50mm -> Capacitors_THT:C_Disc_D4.7mm_W2.5mm_P5.00mm
- C3: footprint Capacitors_THT:CP_Radial_D10.0mm_P2.50mm -> Capacitors_THT:CP_Radial_D8.0mm_P5.00mm
- IC1: value HM62256BLP-7 -> AS6C62256; footprint Housings_DIP:DIP-28_W7.62mm_Socket -> Housings_DIP:DIP-28_W15.24mm_Socket
- IC11: value 74LS153 -> 74HCT251
- IC12, IC4, IC5, IC7, IC8: value 74LS574 -> 74HCT574
- IC13: value 74LS161-wkt -> 74HCT161
- IC14: footprint Housings_DIP:DIP-40_W25.4mm_Socket -> Housings_DIP:DIP-40_W15.24mm_Socket
- IC15: value 74LS139 -> 74HCT139
- IC16: value 74LS138 -> 74HCT138
- IC3: footprint Housings_DIP:DIP-24_W7.62mm_Socket -> Housings_DIP:DIP-24_W15.24mm_Socket
- J1: footprint Connectors:GS3 -> Pin_Headers:Pin_Header_Straight_1x03_Pitch2.54mm
- R1: value 10K -> 20K
- R2: value 10K -> 1K
- U1: value QX14T50B3.6864 -> ECS-100A-035
- moved C3 111.6 mm to (263.7, 67.6)
- moved C10 107.6 mm to (133.6, 76.7), turned to 0 degrees
- moved C12 103.3 mm to (51.8, 72.1), turned to 180 degrees
- moved IC3 97.8 mm to (243.8, 44.7)
- moved C19 96.3 mm to (111.8, 76.7)
- moved C7 95.7 mm to (169.7, 97.5)
- moved R2 81.7 mm to (134.6, 103.1)
- moved IC6 81.0 mm to (178.1, 84.8), turned to 90 degrees
- moved C9 80.4 mm to (229.1, 65.5), turned to 90 degrees
- moved C4 75.8 mm to (175.3, 39.1)
- moved C8 70.0 mm to (254.0, 104.6), turned to 180 degrees
- moved IC10 69.6 mm to (87.9, 39.1)
- moved SW1 65.1 mm to (142.2, 112.3), turned to 90 degrees
- moved IC9 60.3 mm to (77.7, 76.7)
- moved R1 59.8 mm to (134.6, 107.2), turned to 270 degrees
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Connections:
- net IOload renamed ~IOload
- net MEMresult renamed ~MEMresult
- net UARTresult renamed ~UARTresult
- C1 pad 1: Reset -> ~Reset
- C1 pad 2: GND -> Lo
- C10 pad 1: VCC -> Hi
- C10 pad 2: GND -> Lo
- C11 pad 1: VCC -> Hi
- C11 pad 2: GND -> Lo
- C12 pad 1: VCC -> Hi
- C12 pad 2: GND -> Lo
- C13 pad 1: VCC -> Hi
- C13 pad 2: GND -> Lo
- C14 pad 1: VCC -> Hi
- C14 pad 2: GND -> Lo
- C15 pad 1: VCC -> Hi
- C15 pad 2: GND -> Lo
- C16 pad 1: VCC -> Hi
- C16 pad 2: GND -> Lo
- C17 pad 1: VCC -> Hi
- C17 pad 2: GND -> Lo
- C18 pad 1: VCC -> Hi
- C18 pad 2: GND -> Lo
- C19 pad 1: VCC -> Hi
- C19 pad 2: GND -> Lo
- C3 pad 1: VCC -> Hi
- C3 pad 2: GND -> Lo
- C4 pad 1: VCC -> Hi
- C4 pad 2: GND -> Lo
- C5 pad 1: VCC -> Hi
- C5 pad 2: GND -> Lo
- C6 pad 1: VCC -> Hi
- C6 pad 2: GND -> Lo
- C7 pad 1: VCC -> Hi
- C7 pad 2: GND -> Lo
- C8 pad 1: VCC -> Hi
- C8 pad 2: GND -> Lo
- C9 pad 1: VCC -> Hi
- C9 pad 2: GND -> Lo
- IC1 pad 14: GND -> Lo
- IC1 pad 27: MEMload -> ~MEMload
- IC1 pad 28: VCC -> Hi
- IC10 pad 10: GND -> Lo
- IC10 pad 12: Reset -> ~Reset
- IC10 pad 14: PCincr -> ~PCincr
- IC10 pad 15: GND -> Lo
- IC10 pad 17: GND -> Lo
- IC10 pad 18: VCC -> Hi
- IC10 pad 19: ARena -> ~ARena
- IC10 pad 20: VCC -> Hi
- IC11 pad 1: GND -> Zero
- IC11 pad 10: Net-(IC11-Pad10) -> JumpOp1
- IC11 pad 11: Net-(IC11-Pad11) -> JumpOp0
- IC11 pad 12: Net-(IC11-Pad12) -> ~RXready
- IC11 pad 13: Net-(IC11-Pad13) -> ~TXready
- IC11 pad 14: JumpC -> DivByZero
- IC11 pad 15: GND -> Negative
- IC11 pad 16: VCC -> Hi
- IC11 pad 2: JumpZ -> Overflow
- IC11 pad 3: Negative -> Carry
- IC11 pad 4: Zero -> Lo
- IC11 pad 5: Carry -> Net-(IC11-Pad5)
- IC11 pad 6: VCC -> Net-(IC10-Pad9)
- IC11 pad 7: Net-(IC10-Pad9) -> Lo
- IC11 pad 8: (no net) -> Lo
- IC11 pad 9: Net-(IC11-Pad9) -> JumpOp2
- IC12 pad 1: GND -> Lo
- IC12 pad 10: GND -> Lo
- IC12 pad 20: VCC -> Hi
- IC13 pad 1: uSreset -> ~uSreset
- IC13 pad 10: VCC -> Hi
- IC13 pad 16: VCC -> Hi
- IC13 pad 7: VCC -> Hi
- IC13 pad 8: GND -> Lo
- IC13 pad 9: VCC -> Hi
- IC14 pad 1: VCC -> Hi
- IC14 pad 11: GND -> Lo
- IC14 pad 2: GND -> Lo
- IC14 pad 20: GND -> Lo
- IC14 pad 3: Net-(IC14-Pad3) -> ~uSreset
- IC14 pad 30: GND -> Lo
- IC14 pad 34: GND -> Lo
- IC14 pad 35: GND -> Lo
- IC14 pad 36: GND -> Lo
- IC14 pad 37: GND -> Lo
- IC14 pad 39: VCC -> Hi
- IC14 pad 4: uSreset -> ~PCincr
- IC14 pad 40: VCC -> Hi
- IC14 pad 5: PCincr -> ~ARena
- IC14 pad 6: ARena -> JumpOp2
- IC14 pad 7: JumpZ -> JumpOp1
- IC14 pad 8: JumpC -> JumpOp0
- IC15 pad 1: GND -> Lo
- IC15 pad 10: Net-(IC15-Pad10) -> (no net)
- IC15 pad 11: Net-(IC1-Pad20) -> (no net)
- IC15 pad 12: Net-(IC15-Pad12) -> (no net)
- IC15 pad 13: GND -> (no net)
- IC15 pad 14: adr15 -> (no net)
- IC15 pad 15: GND -> (no net)
- IC15 pad 16: VCC -> Hi
- IC15 pad 5: ALUresult -> ~ALUresult
- IC15 pad 8: GND -> Lo
- IC15 pad 9: Net-(IC15-Pad9) -> (no net)
- IC16 pad 10: AHload -> Net-(IC16-Pad10)
- IC16 pad 11: MEMload -> Net-(IC16-Pad11)
- IC16 pad 12: Bload -> Net-(IC16-Pad12)
- IC16 pad 13: Aload -> Net-(IC16-Pad13)
- IC16 pad 14: IRload -> Net-(IC16-Pad14)
- IC16 pad 16: VCC -> Hi
- IC16 pad 4: GND -> Lo
- IC16 pad 5: GND -> Lo
- IC16 pad 6: VCC -> Hi
- IC16 pad 8: GND -> Lo
- IC16 pad 9: ALload -> ~MEMload
- IC2 pad 14: GND -> Lo
- IC2 pad 27: VCC -> Hi
- IC2 pad 28: VCC -> Hi
- IC3 pad 15: VCC -> Hi
- IC3 pad 21: VCC -> Hi
- IC3 pad 22: Net-(IC3-Pad22) -> ~TXready
- IC3 pad 23: Net-(IC3-Pad23) -> ~RXready
- IC3 pad 24: GND -> Lo
- IC3 pad 7: GND -> Lo
- IC4 pad 1: GND -> Lo
- IC4 pad 10: GND -> Lo
- IC4 pad 20: VCC -> Hi
- IC5 pad 1: GND -> Lo
- IC5 pad 10: GND -> Lo
- IC5 pad 20: VCC -> Hi
- IC6 pad 11: ALUresult -> Lo
- IC6 pad 12: GND -> Lo
- IC6 pad 13: GND -> ~ALUresult
- IC6 pad 17: Zero -> Overflow
- IC6 pad 19: Negative -> Zero
- IC6 pad 21: Net-(IC6-Pad21) -> Negative
- IC6 pad 22: VCC -> Hi
- IC6 pad 24: Net-(IC6-Pad24) -> DivByZero
- IC6 pad 31: GND -> Lo
- IC7 pad 1: ARena -> ~ARena
- IC7 pad 10: GND -> Lo
- IC7 pad 20: VCC -> Hi
- IC8 pad 1: ARena -> ~ARena
- IC8 pad 10: GND -> Lo
- IC8 pad 20: VCC -> Hi
- IC9 pad 10: GND -> Lo
- IC9 pad 12: Reset -> ~Reset
- IC9 pad 15: GND -> Lo
- IC9 pad 17: GND -> Lo
- IC9 pad 18: VCC -> Hi
- IC9 pad 19: ARena -> ~ARena
- IC9 pad 20: VCC -> Hi
- J1 pad 3: Net-(C2-Pad1) -> Net-(IC18-Pad3)
- R1 pad 1: VCC -> Hi
- R1 pad 2: Reset -> ~Reset
- R2 pad 1: VCC -> ~Reset
- R2 pad 2: Net-(C2-Pad1) -> Net-(R2-Pad2)
- SW1 pad 3: Reset -> Lo
- SW1 pad 4: GND -> Net-(R2-Pad2)
- SW2 pad 3: Net-(C2-Pad1) -> Lo
- SW2 pad 4: GND -> Net-(C22-Pad2)
- U1 pad 14: VCC -> Hi
- U1 pad 7: GND -> Lo
Routing:
- net Lo: track 0.00 -> 1019.4 mm
- net Hi: track 0.00 -> 719.3 mm, vias 0 -> 1
- net VCC: track 697.1 -> 0.00 mm, vias 5 -> 0
- net ARena: track 297.6 -> 0.00 mm, vias 4 -> 0
- net ~ARena: track 0.00 -> 250.4 mm, vias 0 -> 2
- net PCincr: track 230.4 -> 0.00 mm
- net MEMload: track 145.2 -> 0.00 mm
- net ~Reset: track 0.00 -> 143.0 mm
- net ALUresult: track 141.0 -> 0.00 mm, vias 1 -> 0
- net ~ALUresult: track 0.00 -> 133.2 mm, vias 0 -> 1
- net ~RXready: track 0.00 -> 131.1 mm
- net ~PCincr: track 0.00 -> 129.3 mm
- net ~TXready: track 0.00 -> 125.7 mm
- net ~MEMload: track 0.00 -> 117.4 mm, vias 0 -> 1
- net Reset: track 116.7 -> 0.00 mm
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- added copper zone on B.Cu, net Lo
- added copper zone on F.Cu, net Lo
- removed copper zone on B.Cu, net GND
- removed copper zone on F.Cu, net GND
Other:
- board size 234.9 x 114.3 mm -> 249.9 x 89.4 mm
- net class Power added: clearance 0.3, trace_width 0.381, via_dia 0.7, via_drill 0.5
- rule trace_min: 0.2 -> 0.1524
- board text added: "ALU"
- board text added: "ARhi"
- board text added: "ARlo"
- board text added: "Address bus display"
- board text added: "Areg"
- board text added: "Breg"
- board text added: "CSCvon8 CPU (c) 2019, Warren Toomey"
- board text added: "Clock pulse"
- board text added: "Data bus display"
- board text added: "Data bus reader"
- board text added: "Data bus writer"
- board text added: "Decode ROM"
- board text added: "IR"
- board text added: "IR display"
- board text added: "Inverter"
- board text added: "Jump Logic"
- board text added: "Osc."
- board text added: "Oscillator"
- board text added: "PChi"
- board text added: "PClo"
- board text added: "Phase display"
- board text added: "Pulse"
- board text added: "RAM"
- board text added: "ROM"
- board text added: "Reset"
- board text added: "UART"
- board text added: "uSeq Counter"
- board text added: "v2019/04/10"

Commit message: Updated the schematic and also moved to KiCad 5.
Parts:
- IC15: footprint Housings_DIP:DIP-16_W7.62mm_Socket -> Package_DIP:DIP-16_W7.62mm_Socket
- IC17: value 74LS04 -> 74HCT04
- J1: value GS3 -> Jumper_3_Bridged12; footprint Pin_Headers:Pin_Header_Straight_1x03_Pitch2.54mm -> Connector_PinSocket_2.54mm:PinSocket_1x03_P2.54mm_Vertical
- J2: value DataBus Pin Header -> Data Bus Pin Header; footprint Socket_Strips:Socket_Strip_Straight_1x10_Pitch2.54mm -> Connector_PinSocket_2.54mm:PinSocket_1x10_P2.54mm_Vertical
- J3: value AddressBus Pin Header -> Address Bus Pin Header; footprint Socket_Strips:Socket_Strip_Straight_1x18_Pitch2.54mm -> Connector_PinSocket_2.54mm:PinSocket_1x18_P2.54mm_Vertical
- J4: footprint Socket_Strips:Socket_Strip_Straight_1x06_Pitch2.54mm -> Connector_PinSocket_2.54mm:PinSocket_1x06_P2.54mm_Vertical
- J5: footprint Socket_Strips:Socket_Strip_Straight_1x10_Pitch2.54mm -> Connector_PinSocket_2.54mm:PinSocket_1x10_P2.54mm_Vertical
- moved J2 23.4 mm to (157.0, 62.5), turned to 180 degrees
- moved J5 22.9 mm to (236.7, 62.0), turned to 180 degrees
- moved J4 12.2 mm to (247.4, 87.4), turned to 0 degrees
- moved J1 5.08 mm to (66.5, 104.6), turned to 180 degrees
- moved C12 1.52 mm to (50.3, 72.1)
- moved IC16 1.14 mm to (122.7, 76.5)
- moved C16 1.14 mm to (90.9, 76.2)
- moved IC15 1.14 mm to (100.6, 76.2)
- moved C10 1.14 mm to (134.6, 76.2)
- moved C19 1.14 mm to (112.8, 76.2)
- moved IC9 1.14 mm to (78.7, 76.2)
- moved J3 0.51 mm to (25.4, 91.4)
Connections:
- net Net-(IC10-Pad9) renamed ~PCload
- IC10 pad 13: Clk -> ~Clkbar
- IC10 pad 14: ~PCincr -> Hi
- IC10 pad 15: Lo -> PCincr
- IC10 pad 16: Clk -> ~Clkbar
- IC10 pad 18: Hi -> Lo
- IC13 pad 1: ~uSreset -> ~Reset
- IC13 pad 3: Net-(IC13-Pad3) -> Lo
- IC13 pad 4: Net-(IC13-Pad4) -> Lo
- IC13 pad 5: Net-(IC13-Pad5) -> Lo
- IC13 pad 6: Net-(IC13-Pad6) -> Lo
- IC13 pad 9: Hi -> ~uSreset
- IC14 pad 4: ~PCincr -> PCincr
- IC15 pad 10: (no net) -> Net-(IC15-Pad10)
- IC15 pad 11: (no net) -> ~Clkbar
- IC15 pad 12: (no net) -> Net-(IC15-Pad12)
- IC15 pad 13: (no net) -> Lo
- IC15 pad 14: (no net) -> Clk
- IC15 pad 15: (no net) -> Lo
- IC15 pad 9: (no net) -> Net-(IC15-Pad9)
- IC16 pad 11: Net-(IC16-Pad11) -> ~MEMload
- IC16 pad 4: Lo -> Clk
- IC16 pad 9: ~MEMload -> Net-(IC16-Pad9)
- IC17 pad 11: Net-(IC16-Pad10) -> Net-(IC16-Pad9)
- IC17 pad 9: Net-(IC16-Pad11) -> Net-(IC16-Pad10)
- IC9 pad 13: Clk -> Net-(IC10-Pad11)
- IC9 pad 14: Net-(IC10-Pad11) -> Lo
- IC9 pad 16: Clk -> ~Clkbar
- IC9 pad 18: Hi -> Lo
- J1 pad 1: Net-(J1-Pad1) -> Net-(IC18-Pad3)
- J1 pad 3: Net-(IC18-Pad3) -> Net-(J1-Pad3)
- J2 pad 1: Lo -> d7
- J2 pad 10: d7 -> Lo
- J2 pad 2: Net-(J2-Pad2) -> d6
- J2 pad 3: d0 -> d5
- J2 pad 4: d1 -> d4
- J2 pad 5: d2 -> d3
- J2 pad 6: d3 -> d2
- J2 pad 7: d4 -> d1
- J2 pad 8: d5 -> d0
- J2 pad 9: d6 -> Net-(J2-Pad9)
- J3 pad 1: Lo -> adr15
- J3 pad 10: adr7 -> adr6
- J3 pad 11: adr8 -> adr5
- J3 pad 12: adr9 -> adr4
- J3 pad 13: adr10 -> adr3
- J3 pad 14: adr11 -> adr2
- J3 pad 15: adr12 -> adr1
- J3 pad 16: adr13 -> adr0
- J3 pad 17: adr14 -> Net-(J3-Pad17)
- J3 pad 18: adr15 -> Lo
- J3 pad 2: Net-(J3-Pad2) -> adr14
- J3 pad 3: adr0 -> adr13
- J3 pad 4: adr1 -> adr12
- J3 pad 5: adr2 -> adr11
- J3 pad 6: adr3 -> adr10
- J3 pad 7: adr4 -> adr9
- J3 pad 8: adr5 -> adr8
- J3 pad 9: adr6 -> adr7
- J4 pad 1: Lo -> Net-(IC13-Pad11)
- J4 pad 2: Net-(J4-Pad2) -> Net-(IC13-Pad12)
- J4 pad 3: Net-(IC13-Pad14) -> Net-(IC13-Pad13)
- J4 pad 4: Net-(IC13-Pad13) -> Net-(IC13-Pad14)
- J4 pad 5: Net-(IC13-Pad12) -> Net-(J4-Pad5)
- J4 pad 6: Net-(IC13-Pad11) -> Lo
- J5 pad 1: Lo -> Net-(IC12-Pad12)
- J5 pad 10: Net-(IC12-Pad12) -> Lo
- J5 pad 2: Net-(J5-Pad2) -> Net-(IC12-Pad13)
- J5 pad 3: Net-(IC12-Pad19) -> Net-(IC12-Pad14)
- J5 pad 4: Net-(IC12-Pad18) -> Net-(IC12-Pad15)
- J5 pad 5: Net-(IC12-Pad17) -> Net-(IC12-Pad16)
- J5 pad 6: Net-(IC12-Pad16) -> Net-(IC12-Pad17)
- J5 pad 7: Net-(IC12-Pad15) -> Net-(IC12-Pad18)
- J5 pad 8: Net-(IC12-Pad14) -> Net-(IC12-Pad19)
- J5 pad 9: Net-(IC12-Pad13) -> Net-(J5-Pad9)
- U1 pad 8: Net-(J1-Pad1) -> Net-(J1-Pad3)
Routing:
- net Lo: track 1019.4 -> 0.00 mm
- net Hi: track 719.3 -> 0.00 mm, vias 1 -> 0
- net d3: track 302.5 -> 0.00 mm, vias 1 -> 0
- net d4: track 294.6 -> 0.00 mm, vias 1 -> 0
- net d6: track 293.2 -> 0.00 mm
- net d5: track 278.4 -> 0.00 mm, vias 1 -> 0
- net Clk: track 273.9 -> 0.00 mm, vias 1 -> 0
- net d1: track 268.0 -> 0.00 mm
- net d0: track 260.7 -> 0.00 mm, vias 1 -> 0
- net d2: track 258.4 -> 0.00 mm, vias 2 -> 0
- net ~ARena: track 250.4 -> 0.00 mm, vias 2 -> 0
- net d7: track 242.2 -> 0.00 mm, vias 1 -> 0
- net adr9: track 178.2 -> 0.00 mm, vias 2 -> 0
- net adr15: track 174.9 -> 0.00 mm
- net adr10: track 173.5 -> 0.00 mm, vias 2 -> 0
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- removed copper zone on B.Cu, net Lo
- removed copper zone on F.Cu, net Lo
Other:
- board text added: "v2019/05/05"
- board text removed: "v2019/04/10"

Commit message: Brought the PCB up to date with the new schematic, and tested the RAM with a test program.
Parts:
- added J6: Areg Pin Header, Connector_PinSocket_2.54mm:PinSocket_1x10_P2.54mm_Vertical, F.Cu at (200.3, 62.1)
- added J7: Breg Pin Header, Connector_PinSocket_2.54mm:PinSocket_1x10_P2.54mm_Vertical, F.Cu at (175.3, 62.2)
- IC11: value 74HCT251 -> 74LS251-RESCUE-Schematic; footprint Housings_DIP:DIP-16_W7.62mm_Socket -> Package_DIP:DIP-16_W7.62mm_Socket
- moved J3 53.9 mm to (30.4, 37.7)
- moved IC1 33.4 mm to (72.4, 83.9)
- moved IC2 27.0 mm to (47.0, 84.2)
- moved C12 17.6 mm to (57.1, 88.4), turned to 0 degrees
- moved U1 14.6 mm to (29.5, 107.6)
- moved J5 10.7 mm to (226.1, 62.0)
- moved C4 9.11 mm to (166.9, 35.6)
- moved C11 8.32 mm to (24.1, 84.3)
- moved J1 8.26 mm to (66.5, 112.9)
- moved C21 7.64 mm to (123.3, 112.3), turned to 0 degrees
- moved C18 7.28 mm to (191.8, 35.6)
- moved C13 5.99 mm to (217.2, 35.6)
- moved J2 5.67 mm to (151.3, 62.1)
- moved C14 5.08 mm to (117.9, 39.1)
- moved C15 5.08 mm to (140.2, 39.1)
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Routing:
- net Lo: track 0.00 -> 986.5 mm
- net Hi: track 0.00 -> 691.1 mm
- net d1: track 0.00 -> 294.3 mm, vias 0 -> 1
- net d0: track 0.00 -> 289.0 mm, vias 0 -> 1
- net d3: track 0.00 -> 267.4 mm, vias 0 -> 4
- net d4: track 0.00 -> 261.5 mm
- net d2: track 0.00 -> 253.2 mm, vias 0 -> 2
- net d5: track 0.00 -> 251.2 mm
- net Clk: track 0.00 -> 239.3 mm
- net ~Reset: track 0.00 -> 236.6 mm
- net d7: track 0.00 -> 236.2 mm
- net d6: track 0.00 -> 235.2 mm
- net ~ARena: track 0.00 -> 200.6 mm
- net adr15: track 0.00 -> 199.5 mm, vias 0 -> 1
- net adr9: track 0.00 -> 197.9 mm
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- added copper zone on B.Cu, net Lo
- added copper zone on F.Cu, net Lo
Other:
- net class Default: trace_width 0.25 -> 0.254
- rule via_min_drill: 0.3 -> 0.3048
- rule via_min_size: 0.4 -> 0.508
- board text added: "A reg display"
- board text added: "B reg display"
- board text added: "v2019/05/08"
- board text removed: "v2019/05/05"
